File: dc-scm-rot-jumper-card.kicad_pcb (KiCad board)
At the start: 2 copper layers, 22.2 x 52 mm, 38 parts, among them J1 5019205001

Commit message: Add LICENSE
Parts:
- moved N1 1.25 mm to (145.7, 87.6)
- moved N2 1.19 mm to (139.9, 94.5)
Other:
- board text added: "DC-SCM RoT Jumper Card Rev. 1.1.0"
- board text removed: "Open BMC RoT module Rev. 1.0.1"
Changed lines of the file:
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@@
-(kicad_pcb (version 20171130) (host pcbnew 5.1.9+dfsg1-1~bpo10+1)
+(kicad_pcb (version 20171130) (host pcbnew 5.1.9+dfsg1-1)
   (general
     (thickness 1.6)
@@
   )
   (module dc-scm-rot-jumper-card-footprints:oshw-logo (layer F.Cu)
-    (at 140.98138 94.9664)
+    (at 139.91078 94.455)
     (attr virtual)
     (fp_text reference N2 (at -3.08 -4.76) (layer F.SilkS) hide
@@
   )
   (module dc-scm-rot-jumper-card-footprints:antmicro-logo_scaled_15mm (layer F.Cu)
-    (at 146.85138 88.0214)
+    (at 145.68298 87.5896)
     (attr virtual)
     (fp_text reference N1 (at -7.7 -10.3) (layer F.SilkS) hide
@@
     )
   )
-  (gr_text "Open BMC RoT module \nRev. 1.0.1" (at 143.49638 90.3464) (layer F.Mask)
+  (gr_text "DC-SCM RoT Jumper Card\nRev. 1.1.0" (at 142.32798 89.9146) (layer F.Mask)
     (effects (font (size 0.7 0.7) (thickness 0.15)) (justify left))
   )
-  (gr_text "Open BMC RoT module \nRev. 1.0.1" (at 143.49638 90.3464) (layer F.Cu)
+  (gr_text "DC-SCM RoT Jumper Card\nRev. 1.1.0" (at 142.32798 89.9146) (layer F.Cu)
     (effects (font (size 0.7 0.7) (thickness 0.15)) (justify left))
   )
